Commit message: feat: add end-effector whole-body planning runtime

File: remani_planner/mm_config/meshes/FastArmer/FastArmer.urdf (robot description, URDF)
Before this commit: robot FastArmer, 7 links, 6 joints
Links:
- link base_link: geometry collision mesh filename=package://mm_config/meshes/FastArmer/base_link.STL; visual mesh filename=package://mm_config/meshes/FastArmer/base_link.STL
- link link1: geometry collision mesh filename=package://mm_config/meshes/FastArmer/link1.STL; visual mesh filename=package://mm_config/meshes/FastArmer/link1.STL
- link link2: geometry collision mesh filename=package://mm_config/meshes/FastArmer/link2.STL; visual mesh filename=package://mm_config/meshes/FastArmer/link2.STL
- link link3: geometry collision mesh filename=package://mm_config/meshes/FastArmer/link3.STL; visual mesh filename=package://mm_config/meshes/FastArmer/link3.STL
- link link4: geometry collision mesh filename=package://mm_config/meshes/FastArmer/link4.STL; visual mesh filename=package://mm_config/meshes/FastArmer/link4.STL
- link link5: geometry collision mesh filename=package://mm_config/meshes/FastArmer/link5.STL; visual mesh filename=package://mm_config/meshes/FastArmer/link5.STL
- link link6: geometry collision mesh filename=package://mm_config/meshes/FastArmer/link6.STL; visual mesh filename=package://mm_config/meshes/FastArmer/link6.STL
